File: v0001/mobile-lipo-charger-v0001.sch (EAGLE design)
At the start: 38 parts, among them IC1 AD8610MR, IC2 STM32F401VBT, IC3 AD8610MR, SW1 DHT-4235A

Commit message: Added 3.3V rail
Added the 3.3V rail switching supply
Parts:
- added C21: 100n, common:CAP0603L3
- added C22, C23: 10u, common:CAP1206L3
- added C24, C25, C26: 22u, common:CAP0603L3
- added L1: 2.2uH, common:INDUCTOR10X10
- added R10: 10k, common:RES0402L3
- added R9: 33.2k, common:RES0402L3
- added U3: 3.3V, common:TPS564201
Connections:
- new net SW: C21.1, L1.1, U3.SW
- new net VBST: C21.2, U3.VBST
- new net VFB: R10.2, R9.1, U3.VFB
- net BATT+: now also C22.1, C23.1, U3.EN, U3.VIN
- net GND: now also C22.2, C23.2, C24.2, C25.2, C26.2, R10.1, U3.GND
- net VDD: now also C24.1, C25.1, C26.1, L1.2, R9.2
Changed lines of the file:
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@@
 <part name="GND27" library="SparkFun-Aesthetics" deviceset="GND" device=""/>
 <part name="SUPPLY4" library="SparkFun-PowerSymbols" library_urn="urn:adsk.eagle:library:530" deviceset="VDD" device=""/>
+<part name="U3" library="common" deviceset="TPS564201" device="" value="3.3V"/>
+<part name="C21" library="common" deviceset="CAP" device="0603L3" value="100n"/>
+<part name="R9" library="common" deviceset="RES" device="0402L3" value="33.2k"/>
+<part name="R10" library="common" deviceset="RES" device="0402L3" value="10k"/>
+<part name="C22" library="common" deviceset="CAP" device="1206L3" value="10u"/>
+<part name="C23" library="common" deviceset="CAP" device="1206L3" value="10u"/>
+<part name="GND28" library="SparkFun-Aesthetics" deviceset="GND" device=""/>
+<part name="L1" library="common" deviceset="INDUCTOR" device="10X10" value="2.2uH"/>
+<part name="SUPPLY5" library="SparkFun-PowerSymbols" library_urn="urn:adsk.eagle:library:530" deviceset="VDD" device=""/>
+<part name="C24" library="common" deviceset="CAP" device="0603L3" value="22u"/>
+<part name="C25" library="common" deviceset="CAP" device="0603L3" value="22u"/>
+<part name="C26" library="common" deviceset="CAP" device="0603L3" value="22u"/>
 </parts>
 <sheets>
@@
 </plain>
 <instances>
+<instance part="U3" gate="G$1" x="0" y="0" smashed="yes">
+<attribute name="NAME" x="-10.16" y="8.636" size="1.778" layer="95"/>
+<attribute name="VALUE" x="-10.16" y="-10.16" size="1.778" layer="96"/>
+</instance>
+<instance part="C21" gate="G$1" x="27.94" y="0" smashed="yes">
+<attribute name="NAME" x="28.956" y="0.508" size="1.778" layer="95"/>
+<attribute name="VALUE" x="28.956" y="-4.826" size="1.778" layer="96"/>
+</instance>
+<instance part="R9" gate="G$1" x="45.72" y="0" smashed="yes" rot="R90">
+<attribute name="NAME" x="44.196" y="-2.54" size="1.778" layer="95" rot="R90"/>
+<attribute name="VALUE" x="48.768" y="-2.54" size="1.778" layer="96" rot="R90"/>
+</instance>
+<instance part="R10" gate="G$1" x="45.72" y="-10.16" smashed="yes" rot="R90">
+<attribute name="NAME" x="44.196" y="-12.7" size="1.778" layer="95" rot="R90"/>
+<attribute name="VALUE" x="48.768" y="-12.7" size="1.778" layer="96" rot="R90"/>
+</instance>
+<instance part="C22" gate="G$1" x="-27.94" y="0" smashed="yes">
+<attribute name="NAME" x="-26.924" y="0.508" size="1.778" layer="95"/>
+<attribute name="VALUE" x="-26.924" y="-4.826" size="1.778" layer="96"/>
+</instance>
+<instance part="C23" gate="G$1" x="-35.56" y="0" smashed="yes">
+<attribute name="NAME" x="-34.544" y="0.508" size="1.778" layer="95"/>
+<attribute name="VALUE" x="-34.544" y="-4.826" size="1.778" layer="96"/>
+</instance>
+<instance part="GND28" gate="1" x="2.54" y="-20.32" smashed="yes">
+<attribute name="VALUE" x="0" y="-22.86" size="1.778" layer="96"/>
+</instance>
+<instance part="L1" gate="G$1" x="38.1" y="5.08" smashed="yes">
+<attribute name="NAME" x="35.56" y="6.35" size="1.778" layer="95"/>
+<attribute name="VALUE" x="35.56" y="1.524" size="1.778" layer="96"/>
+</instance>
+<instance part="SUPPLY5" gate="VDD" x="45.72" y="7.62" smashed="yes">
+<attribute name="VALUE" x="45.72" y="10.414" size="1.778" layer="96" align="bottom-center"/>
+</instance>
+<instance part="C24" gate="G$1" x="55.88" y="0" smashed="yes">
+<attribute name="NAME" x="56.896" y="0.508" size="1.778" layer="95"/>
+<attribute name="VALUE" x="56.896" y="-4.826" size="1.778" layer="96"/>
+</instance>
+<instance part="C25" gate="G$1" x="63.5" y="0" smashed="yes">
+<attribute name="NAME" x="64.516" y="0.508" size="1.778" layer="95"/>
+<attribute name="VALUE" x="64.516" y="-4.826" size="1.778" layer="96"/>
+</instance>
+<instance part="C26" gate="G$1" x="71.12" y="0" smashed="yes">
+<attribute name="NAME" x="72.136" y="0.508" size="1.778" layer="95"/>
+<attribute name="VALUE" x="72.136" y="-4.826" size="1.778" layer="96"/>
+</instance>
 </instances>
 <busses>
 </busses>
 <nets>
+<net name="SW" class="0">
+<segment>
+<pinref part="U3" gate="G$1" pin="SW"/>
+<pinref part="C21" gate="G$1" pin="1"/>
+<wire x1="15.24" y1="5.08" x2="27.94" y2="5.08" width="0.1524" layer="91"/>
+<wire x1="27.94" y1="5.08" x2="27.94" y2="2.54" width="0.1524" layer="91"/>
+<pinref part="L1" gate="G$1" pin="1"/>
+<wire x1="27.94" y1="5.08" x2="35.56" y2="5.08" width="0.1524" layer="91"/>
+<junction x="27.94" y="5.08"/>
+<label x="17.78" y="5.08" size="1.778" layer="95"/>
+</segment>
+</net>
+<net name="VBST" class="0">
+<segment>
+<pinref part="U3" gate="G$1" pin="VBST"/>
+<wire x1="15.24" y1="2.54" x2="22.86" y2="2.54" width="0.1524" layer="91"/>
+<wire x1="22.86" y1="2.54" x2="22.86" y2="-7.62" width="0.1524" layer="91"/>
+<pinref part="C21" gate="G$1" pin="2"/>
+<wire x1="22.86" y1="-7.62" x2="27.94" y2="-7.62" width="0.1524" layer="91"/>
+<wire x1="27.94" y1="-7.62" x2="27.94" y2="-5.08" width="0.1524" layer="91"/>
+<label x="17.78" y="2.54" size="1.778" layer="95"/>
+</segment>
+</net>
+<net name="VFB" class="0">
+<segment>
+<pinref part="R9" gate="G$1" pin="1"/>
+<pinref part="R10" gate="G$1" pin="2"/>
+<wire x1="45.72" y1="-2.54" x2="45.72" y2="-5.08" width="0.1524" layer="91"/>
+<wire x1="45.72" y1="-5.08" x2="45.72" y2="-7.62" width="0.1524" layer="91"/>
+<wire x1="45.72" y1="-5.08" x2="35.56" y2="-5.08" width="0.1524" layer="91"/>
+<wire x1="35.56" y1="-5.08" x2="35.56" y2="-10.16" width="0.1524" layer="91"/>
+<junction x="45.72" y="-5.08"/>
+<wire x1="35.56" y1="-10.16" x2="20.32" y2="-10.16" width="0.1524" layer="91"/>
+<wire x1="20.32" y1="-10.16" x2="20.32" y2="-2.54" width="0.1524" layer="91"/>
+<pinref part="U3" gate="G$1" pin="VFB"/>
+<wire x1="20.32" y1="-2.54" x2="15.24" y2="-2.54" width="0.1524" layer="91"/>
+<label x="17.78" y="-2.54" size="1.778" layer="95"/>
+</segment>
+</net>
+<net name="BATT+" class="0">
+<segment>
+<pinref part="U3" gate="G$1" pin="VIN"/>
+<pinref part="C22" gate="G$1" pin="1"/>
+<wire x1="-15.24" y1="5.08" x2="-17.78" y2="5.08" width="0.1524" layer="91"/>
+<wire x1="-17.78" y1="5.08" x2="-27.94" y2="5.08" width="0.1524" layer="91"/>
+<wire x1="-27.94" y1="5.08" x2="-27.94" y2="2.54" width="0.1524" layer="91"/>
+<pinref part="C23" gate="G$1" pin="1"/>
+<wire x1="-27.94" y1="5.08" x2="-35.56" y2="5.08" width="0.1524" layer="91"/>
+<wire x1="-35.56" y1="5.08" x2="-35.56" y2="2.54" width="0.1524" layer="91"/>
+<junction x="-27.94" y="5.08"/>
+<pinref part="U3" gate="G$1" pin="EN"/>
+<wire x1="-17.78" y1="5.08" x2="-17.78" y2="2.54" width="0.1524" layer="91"/>
+<wire x1="-17.78" y1="2.54" x2="-15.24" y2="2.54" width="0.1524" layer="91"/>
+<junction x="-17.78" y="5.08"/>
+<wire x1="-43.18" y1="5.08" x2="-35.56" y2="5.08" width="0.1524" layer="91"/>
+<junction x="-35.56" y="5.08"/>
+<label x="-43.18" y="5.08" size="1.778" layer="95"/>
+</segment>
+</net>
+<net name="GND" class="0">
+<segment>
+<pinref part="U3" gate="G$1" pin="GND"/>
+<wire x1="15.24" y1="-5.08" x2="17.78" y2="-5.08" width="0.1524" layer="91"/>
+<wire x1="17.78" y1="-5.08" x2="17.78" y2="-15.24" width="0.1524" layer="91"/>
+<pinref part="R10" gate="G$1" pin="1"/>
+<wire x1="17.78" y1="-15.24" x2="45.72" y2="-15.24" width="0.1524" layer="91"/>
+<wire x1="45.72" y1="-15.24" x2="45.72" y2="-12.7" width="0.1524" layer="91"/>
+<pinref part="C22" gate="G$1" pin="2"/>
+<wire x1="-27.94" y1="-5.08" x2="-27.94" y2="-15.24" width="0.1524" layer="91"/>
+<wire x1="-27.94" y1="-15.24" x2="2.54" y2="-15.24" width="0.1524" layer="91"/>
+<junction x="17.78" y="-15.24"/>
+<pinref part="C23" gate="G$1" pin="2"/>
+<wire x1="2.54" y1="-15.24" x2="17.78" y2="-15.24" width="0.1524" layer="91"/>
+<wire x1="-35.56" y1="-5.08" x2="-35.56" y2="-15.24" width="0.1524" layer="91"/>
+<wire x1="-35.56" y1="-15.24" x2="-27.94" y2="-15.24" width="0.1524" layer="91"/>
+<junction x="-27.94" y="-15.24"/>
+<pinref part="GND28" gate="1" pin="GND"/>
+<wire x1="2.54" y1="-17.78" x2="2.54" y2="-15.24" width="0.1524" layer="91"/>
+<junction x="2.54" y="-15.24"/>
+<pinref part="C24" gate="G$1" pin="2"/>
+<wire x1="45.72" y1="-15.24" x2="55.88" y2="-15.24" width="0.1524" layer="91"/>
+<wire x1="55.88" y1="-15.24" x2="55.88" y2="-5.08" width="0.1524" layer="91"/>
+<junction x="45.72" y="-15.24"/>
+<pinref part="C25" gate="G$1" pin="2"/>
+<wire x1="55.88" y1="-15.24" x2="63.5" y2="-15.24" width="0.1524" layer="91"/>
+<wire x1="63.5" y1="-15.24" x2="63.5" y2="-5.08" width="0.1524" layer="91"/>
+<junction x="55.88" y="-15.24"/>
+<pinref part="C26" gate="G$1" pin="2"/>
+<wire x1="63.5" y1="-15.24" x2="71.12" y2="-15.24" width="0.1524" layer="91"/>
+<wire x1="71.12" y1="-15.24" x2="71.12" y2="-5.08" width="0.1524" layer="91"/>
+<junction x="63.5" y="-15.24"/>
+</segment>
+</net>
+<net name="VDD" class="0">
+<segment>
+<pinref part="R9" gate="G$1" pin="2"/>
+<wire x1="45.72" y1="5.08" x2="45.72" y2="2.54" width="0.1524" layer="91"/>
+<pinref part="L1" gate="G$1" pin="2"/>
+<wire x1="40.64" y1="5.08" x2="45.72" y2="5.08" width="0.1524" layer="91"/>
+<pinref part="SUPPLY5" gate="VDD" pin="VDD"/>
+<wire x1="45.72" y1="7.62" x2="45.72" y2="5.08" width="0.1524" layer="91"/>
+<junction x="45.72" y="5.08"/>
+<pinref part="C24" gate="G$1" pin="1"/>
+<wire x1="45.72" y1="5.08" x2="55.88" y2="5.08" width="0.1524" layer="91"/>
+<wire x1="55.88" y1="5.08" x2="55.88" y2="2.54" width="0.1524" layer="91"/>
+<pinref part="C25" gate="G$1" pin="1"/>
+<wire x1="55.88" y1="5.08" x2="63.5" y2="5.08" width="0.1524" layer="91"/>
+<wire x1="63.5" y1="5.08" x2="63.5" y2="2.54" width="0.1524" layer="91"/>
+<junction x="55.88" y="5.08"/>
+<pinref part="C26" gate="G$1" pin="1"/>
+<wire x1="63.5" y1="5.08" x2="71.12" y2="5.08" width="0.1524" layer="91"/>
+<wire x1="71.12" y1="5.08" x2="71.12" y2="2.54" width="0.1524" layer="91"/>
+<junction x="63.5" y="5.08"/>
+</segment>
+</net>
 </nets>
 </sheet>

Commit message: Minor Changes
Made minor changes to the polygons for the charger chips
Parts:
- added C27: 100n, common:CAP0603L3
- added C28, C29: 10u, common:CAP1206L3
- added C30, C31: 22u, common:CAP0603L3
- added L2: 3.3uH, common:INDUCTOR10X10
- added R11: 75k, common:RES0402L3
- added R12: 10k, common:RES0402L3
- added U4: 3.3V, common:TPS564201
Connections:
- new net SW2: C27.1, L2.1, U4.SW
- new net VBST2: C27.2, U4.VBST
- new net VFB2: R11.1, R12.2, U4.VFB
- new net VIN_CHARGER: C1.1, C16.1, C30.1, C31.1, L2.2, R11.2, U1.VIN, U2.VIN
- net BATT+: now also C28.1, C29.1, U4.EN, U4.VIN; no longer C1.1, C16.1, U1.VIN, U2.VIN
- net GND: now also C28.2, C29.2, C30.2, C31.2, R12.1, U4.GND
